File: Redoubot/connectors.kicad_sch (KiCad schematic)
At the start: 12 parts, among them J1 Connecteur batterie, J10 HM_10_BLE_Module, J11 DFPlayer_Left, J12 DFPlayer_Right, J2 Motor_Left, J3 Motor_Right, J4 Servo_Left, J5 MPU-6050, J6 APDS9960, J7 VL53L0CXV0DH - TOF, J8 Servo_Right, J9 Neopixel

Commit message: added the footprints for the connectors
Parts:
- J1: footprint (none) -> Connector_JST:JST_XH_B2B-XH-A_1x02_P2.50mm_Vertical
- J10, J6: footprint (none) -> Connector_PinSocket_2.54mm:PinSocket_1x06_P2.54mm_Vertical
- J11, J12, J5: footprint (none) -> Connector_PinSocket_2.54mm:PinSocket_1x08_P2.54mm_Vertical
- J2, J3: footprint (none) -> Connector_JST:JST_ZH_B2B-ZR_1x02_P1.50mm_Vertical
- J4: footprint Package_BGA:BGA-256_17.0x17.0mm_Layout16x16_P1.0mm_Ball0.5mm_Pad0.4mm_NSMD -> Connector_PinHeader_2.54mm:PinHeader_1x03_P2.54mm_Vertical
- J8, J9: footprint (none) -> Connector_PinHeader_2.54mm:PinHeader_1x03_P2.54mm_Vertical
Changed lines of the file:
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@@
 			)
 		)
-		(property "Footprint" ""
+		(property "Footprint" "Connector_PinSocket_2.54mm:PinSocket_1x08_P2.54mm_Vertical"
 			(at 107.95 96.52 0)
 			(hide yes)
@@
 			)
 		)
-		(property "Footprint" "Package_BGA:BGA-256_17.0x17.0mm_Layout16x16_P1.0mm_Ball0.5mm_Pad0.4mm_NSMD"
+		(property "Footprint" "Connector_PinHeader_2.54mm:PinHeader_1x03_P2.54mm_Vertical"
 			(at 133.35 66.04 0)
 			(hide yes)
@@
 			)
 		)
-		(property "Footprint" ""
+		(property "Footprint" "Connector_PinSocket_2.54mm:PinSocket_1x08_P2.54mm_Vertical"
 			(at 170.18 120.65 0)
 			(hide yes)
@@
 			)
 		)
-		(property "Footprint" ""
+		(property "Footprint" "Connector_JST:JST_ZH_B2B-ZR_1x02_P1.50mm_Vertical"
 			(at 107.95 63.5 0)
 			(hide yes)
@@
 			)
 		)
-		(property "Footprint" ""
+		(property "Footprint" "Connector_PinHeader_2.54mm:PinHeader_1x03_P2.54mm_Vertical"
 			(at 176.53 66.04 0)
 			(hide yes)
@@
 			)
 		)
-		(property "Footprint" ""
+		(property "Footprint" "Connector_PinSocket_2.54mm:PinSocket_1x08_P2.54mm_Vertical"
 			(at 137.16 120.65 0)
 			(hide yes)
@@
 			)
 		)
-		(property "Footprint" ""
+		(property "Footprint" "Connector_PinSocket_2.54mm:PinSocket_1x06_P2.54mm_Vertical"
 			(at 82.55 121.92 0)
 			(hide yes)
@@
 			)
 		)
-		(property "Footprint" ""
+		(property "Footprint" "Connector_PinSocket_2.54mm:PinSocket_1x06_P2.54mm_Vertical"
 			(at 82.55 93.98 0)
 			(hide yes)
@@
 			)
 		)
-		(property "Footprint" ""
+		(property "Footprint" "Connector_PinHeader_2.54mm:PinHeader_1x03_P2.54mm_Vertical"
 			(at 133.35 91.44 0)
 			(hide yes)
@@
 			)
 		)
-		(property "Footprint" ""
+		(property "Footprint" "Connector_JST:JST_XH_B2B-XH-A_1x02_P2.50mm_Vertical"
 			(at 111.76 45.72 0)
 			(hide yes)
@@
 			)
 		)
-		(property "Footprint" ""
+		(property "Footprint" "Connector_JST:JST_ZH_B2B-ZR_1x02_P1.50mm_Vertical"
 			(at 107.95 73.66 0)
 			(hide yes)

Commit message: fixed the footprint for the connector of the VL53
Parts:
- J7: footprint Package_BGA:BGA-256_17.0x17.0mm_Layout16x16_P1.0mm_Ball0.5mm_Pad0.4mm_NSMD -> Connector_PinSocket_2.54mm:PinSocket_1x06_P2.54mm_Vertical
Changed lines of the file:
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@@
 			)
 		)
-		(property "Footprint" "Package_BGA:BGA-256_17.0x17.0mm_Layout16x16_P1.0mm_Ball0.5mm_Pad0.4mm_NSMD"
+		(property "Footprint" "Connector_PinSocket_2.54mm:PinSocket_1x06_P2.54mm_Vertical"
 			(at 82.55 68.58 0)
 			(hide yes)

Commit message: feat: added usb_c charging + flashing, added +3.3V generation, added HM10 & DFMini Support, wired everything and modified ioc accordingly
Parts:
- added J14: Speaker, Package_DFN_QFN:QFN-20-1EP_5x5mm_P0.65mm_EP3.35x3.35mm, symbol Connector:Conn_01x02_Pin
Connections:
- net SPK1: now also J14.1 (Pin_1)
- net SPK2: now also J14.2 (Pin_2)
Changed lines of the file:
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@@
+	(wire
+		(pts
+			(xy 147.32 115.57) (xy 142.24 115.57)
+		)
+		(stroke
+			(width 0)
+			(type default)
+		)
+	)
 	(wire
 		(pts
@@
 	(wire
 		(pts
+			(xy 147.32 130.81) (xy 142.24 130.81)
+		)
+		(stroke
+			(width 0)
+			(type default)
+		)
+	)
+	(wire
+		(pts
 			(xy 115.57 91.44) (xy 113.03 91.44)
 		)
@@
 	(wire
 		(pts
+			(xy 179.07 113.03) (xy 175.26 113.03)
+		)
+		(stroke
+			(width 0)
+			(type default)
+		)
+	)
+	(wire
+		(pts
 			(xy 90.17 93.98) (xy 87.63 93.98)
 		)
@@
 	(wire
 		(pts
+			(xy 147.32 113.03) (xy 142.24 113.03)
+		)
+		(stroke
+			(width 0)
+			(type default)
+		)
+	)
+	(wire
+		(pts
 			(xy 87.63 127) (xy 90.17 127)
 		)
@@
 	(wire
 		(pts
+			(xy 147.32 118.11) (xy 142.24 118.11)
+		)
+		(stroke
+			(width 0)
+			(type default)
+		)
+	)
+	(wire
+		(pts
 			(xy 90.17 96.52) (xy 87.63 96.52)
 		)
@@
 	(wire
 		(pts
+			(xy 207.01 115.57) (xy 203.2 115.57)
+		)
+		(stroke
+			(width 0)
+			(type default)
+		)
+	)
+	(wire
+		(pts
 			(xy 87.63 71.12) (xy 90.17 71.12)
 		)
@@
 	(wire
 		(pts
+			(xy 179.07 128.27) (xy 175.26 128.27)
+		)
+		(stroke
+			(width 0)
+			(type default)
+		)
+	)
+	(wire
+		(pts
 			(xy 90.17 63.5) (xy 87.63 63.5)
 		)
@@
 	(wire
 		(pts
+			(xy 147.32 128.27) (xy 142.24 128.27)
+		)
+		(stroke
+			(width 0)
+			(type default)
+		)
+	)
+	(wire
+		(pts
 			(xy 90.17 101.6) (xy 87.63 101.6)
 		)
@@
 	(wire
 		(pts
+			(xy 147.32 125.73) (xy 142.24 125.73)
+		)
+		(stroke
+			(width 0)
+			(type default)
+		)
+	)
+	(wire
+		(pts
 			(xy 87.63 73.66) (xy 90.17 73.66)
 		)
@@
 	(wire
 		(pts
+			(xy 207.01 113.03) (xy 203.2 113.03)
+		)
+		(stroke
+			(width 0)
+			(type default)
+		)
+	)
+	(wire
+		(pts
 			(xy 181.61 63.5) (xy 185.42 63.5)
 		)
@@
 			(width 0)
 			(type default)
+		)
+	)
+	(label "SPK2"
+		(at 207.01 115.57 0)
+		(effects
+			(font
+				(size 1.27 1.27)
+			)
+			(justify left bottom)
+		)
+	)
+	(label "SPK1"
+		(at 207.01 113.03 0)
+		(effects
+			(font
+				(size 1.27 1.27)
+			)
+			(justify left bottom)
+		)
+	)
+	(label "SPK2"
+		(at 147.32 130.81 0)
+		(effects
+			(font
+				(size 1.27 1.27)
+			)
+			(justify left bottom)
+		)
+	)
+	(label "SPK1"
+		(at 147.32 125.73 0)
+		(effects
+			(font
+				(size 1.27 1.27)
+			)
+			(justify left bottom)
 		)
 	)
@@
 		)
 	)
-	(hierarchical_label "SPK2"
-		(shape input)
-		(at 142.24 130.81 0)
-		(effects
-			(font
-				(size 1.27 1.27)
-			)
-			(justify left)
-		)
-	)
 	(hierarchical_label "SDA_ADA"
 		(shape bidirectional)
@@
 	(hierarchical_label "VCC_DF"
 		(shape input)
-		(at 142.24 113.03 0)
+		(at 147.32 113.03 0)
 		(effects
 			(font
@@
 	(hierarchical_label "GND"
 		(shape input)
-		(at 175.26 128.27 0)
+		(at 179.07 128.27 0)
 		(effects
 			(font
@@
 	)
 	(hierarchical_label "TXD_HM10"
-		(shape input)
+		(shape output)
 		(at 90.17 124.46 0)
 		(effects
@@
 	)
 	(hierarchical_label "TX_DF"
-		(shape input)
-		(at 142.24 118.11 0)
+		(shape output)
+		(at 147.32 118.11 0)
 		(effects
 			(font
@@
 	)
 	(hierarchical_label "BUSY"
-		(shape input)
-		(at 175.26 113.03 0)
+		(shape output)
+		(at 179.07 113.03 0)
 		(effects
 			(font
@@
 		)
 	)
-	(hierarchical_label "SPK1"
-		(shape input)
-		(at 142.24 125.73 0)
-		(effects
-			(font
-				(size 1.27 1.27)
-			)
-			(justify left)
-		)
-	)
 	(hierarchical_label "STATE_HM10"
-		(shape input)
+		(shape output)
 		(at 90.17 116.84 0)
 		(effects
@@
 	(hierarchical_label "RX_DF"
 		(shape input)
-		(at 142.24 115.57 0)
+		(at 147.32 115.57 0)
 		(effects
 			(font
@@
 	(hierarchical_label "GND"
 		(shape input)
-		(at 142.24 128.27 0)
+		(at 147.32 128.27 0)
 		(effects
 			(font
@@
 					(unit 1)
 				)
+			)
+		)
+	)
+	(symbol
+		(lib_id "Connector:Conn_01x02_Pin")
+		(at 198.12 113.03 0)
+		(unit 1)
+		(body_style 1)
+		(exclude_from_sim no)
+		(in_bom yes)
+		(on_board yes)
+		(in_pos_files yes)
+		(dnp no)
+		(fields_autoplaced yes)
+		(property "Reference" "J14"
+			(at 198.755 107.95 0)
+			(show_name no)
+			(do_not_autoplace no)
+			(effects
+				(font
+					(size 1.27 1.27)
+				)
+			)
+		)
+		(property "Value" "Speaker"
+			(at 198.755 110.49 0)
+			(show_name no)
+			(do_not_autoplace no)
+			(effects
+				(font
+					(size 1.27 1.27)
+				)
+			)
+		)
+		(property "Footprint" "Package_DFN_QFN:QFN-20-1EP_5x5mm_P0.65mm_EP3.35x3.35mm"
+			(at 198.12 113.03 0)
+			(hide yes)
+			(show_name no)
+			(do_not_autoplace no)
+			(effects
+				(font
+					(size 1.27 1.27)
+				)
+			)
+		)
+		(property "Datasheet" ""
+			(at 198.12 113.03 0)
+			(hide yes)
+			(show_name no)
+			(do_not_autoplace no)
+			(effects
+				(font
+					(size 1.27 1.27)
+				)
+			)
+		)
+		(property "Description" "Generic connector, single row, 01x02, script generated"
+			(at 198.12 113.03 0)
+			(hide yes)
+			(show_name no)
+			(do_not_autoplace no)
+			(effects
+				(font
+					(size 1.27 1.27)
+				)
+			)
+		)
+		(pin "2"
+		)
+		(pin "1"
+		)
+		(instances
+			(project "Redoubot"
+				(path "/43131b41-4104-4cd6-9c2f-4d5da1687300/6319d978-6c6a-440c-b0e5-feb4687d4119"
+					(reference "J14")
+					(unit 1)
+				)
