File: Redoubot/usb_c.kicad_sch (KiCad schematic)
At the start: 4 parts, among them J13 USB_C_Receptacle_USB2.0_16P, U6 USBLC6-2SC6

Commit message: replaced the footprints for resistors with 0402 variants
Parts:
- R5, R6: footprint Resistor_SMD:R_0805_2012Metric -> Resistor_SMD:R_0402_1005Metric
Changed lines of the file:
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@@
 			)
 		)
-		(property "Footprint" "Resistor_SMD:R_0805_2012Metric"
+		(property "Footprint" "Resistor_SMD:R_0402_1005Metric"
 			(at 69.85 39.37 0)
 			(hide yes)
@@
 			)
 		)
-		(property "Footprint" "Resistor_SMD:R_0805_2012Metric"
+		(property "Footprint" "Resistor_SMD:R_0402_1005Metric"
 			(at 69.85 34.29 0)
 			(hide yes)
