File: Redoubot/drivers.kicad_sch (KiCad schematic)
At the start: 0 parts

Commit message: feat: motor driver wired in parallel mode
Parts:
- added C1: 0.1µF, symbol Device:C_Small
- added C2: 10µF, symbol Device:C_Polarized_Small
- added C3: 2.2µF, symbol Device:C_Small
- added R1: 200m, symbol Device:R_Small_US
- added U2: DRV8833PWP, Package_SO:HTSSOP-16-1EP_4.4x5mm_P0.65mm_EP3.4x5mm_Mask2.46x2.31mm_ThermalVias, symbol Driver_Motor:DRV8833PWP
Connections:
- new net: C1.2, U2.11 (VCP)
- new net: R1.2, U2.3 (AISEN), U2.6 (BISEN)
- new net: C3.1, U2.14 (VINT)
- new net GND: C2.2, C3.2, R1.1, U2.13 (GND), U2.17 (GND)
- new net GPIO_NSLEEP: U2.1 (~{SLEEP})
- new net M1: U2.2 (AOUT1), U2.7 (BOUT1)
- new net M2: U2.4 (AOUT2), U2.5 (BOUT2)
- new net PWM_IN1: U2.16 (AIN1), U2.9 (BIN1)
- new net PWM_IN2: U2.10 (BIN2), U2.15 (AIN2)
- new net VM: C1.1, C2.1, U2.12 (VM)
- no-connect marks 0 -> 1
Other:
- note added: "Low = Sleep; High = Run"

Commit message: feat: added all remaining connectors & finished putting values on components
Connections:
- net M1 renamed M+
- net M2 renamed M-
Changed lines of the file:
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@@
 		)
 	)
-	(hierarchical_label "M1"
-		(shape input)
+	(hierarchical_label "M+"
+		(shape output)
 		(at 129.54 57.15 0)
 		(effects
@@
 		)
 	)
-	(hierarchical_label "M2"
-		(shape input)
+	(hierarchical_label "M-"
+		(shape output)
 		(at 129.54 64.77 0)
 		(effects
@@
 		(instances
 			(project "Redoubot"
+				(path "/43131b41-4104-4cd6-9c2f-4d5da1687300/089490fe-51aa-455e-8e68-3144de50c1de"
+					(reference "C8")
+					(unit 1)
+				)
 				(path "/43131b41-4104-4cd6-9c2f-4d5da1687300/b7c7d3a9-6fc5-4331-a1be-dcf952831da1"
 					(reference "C1")
@@
 		(instances
 			(project "Redoubot"
+				(path "/43131b41-4104-4cd6-9c2f-4d5da1687300/089490fe-51aa-455e-8e68-3144de50c1de"
+					(reference "R5")
+					(unit 1)
+				)
 				(path "/43131b41-4104-4cd6-9c2f-4d5da1687300/b7c7d3a9-6fc5-4331-a1be-dcf952831da1"
 					(reference "R1")
@@
 		(instances
 			(project "Redoubot"
+				(path "/43131b41-4104-4cd6-9c2f-4d5da1687300/089490fe-51aa-455e-8e68-3144de50c1de"
+					(reference "#PWR09")
+					(unit 1)
+				)
 				(path "/43131b41-4104-4cd6-9c2f-4d5da1687300/b7c7d3a9-6fc5-4331-a1be-dcf952831da1"
 					(reference "#PWR02")
@@
 		(instances
 			(project "Redoubot"
+				(path "/43131b41-4104-4cd6-9c2f-4d5da1687300/089490fe-51aa-455e-8e68-3144de50c1de"
+					(reference "U3")
+					(unit 1)
+				)
 				(path "/43131b41-4104-4cd6-9c2f-4d5da1687300/b7c7d3a9-6fc5-4331-a1be-dcf952831da1"
 					(reference "U2")
@@
 		(instances
 			(project "Redoubot"
+				(path "/43131b41-4104-4cd6-9c2f-4d5da1687300/089490fe-51aa-455e-8e68-3144de50c1de"
+					(reference "C9")
+					(unit 1)
+				)
 				(path "/43131b41-4104-4cd6-9c2f-4d5da1687300/b7c7d3a9-6fc5-4331-a1be-dcf952831da1"
 					(reference "C3")
@@
 		(instances
 			(project "Redoubot"
+				(path "/43131b41-4104-4cd6-9c2f-4d5da1687300/089490fe-51aa-455e-8e68-3144de50c1de"
+					(reference "#PWR010")
+					(unit 1)
+				)
 				(path "/43131b41-4104-4cd6-9c2f-4d5da1687300/b7c7d3a9-6fc5-4331-a1be-dcf952831da1"
 					(reference "#PWR03")
@@
 		(instances
 			(project "Redoubot"
+				(path "/43131b41-4104-4cd6-9c2f-4d5da1687300/089490fe-51aa-455e-8e68-3144de50c1de"
+					(reference "#PWR023")
+					(unit 1)
+				)
 				(path "/43131b41-4104-4cd6-9c2f-4d5da1687300/b7c7d3a9-6fc5-4331-a1be-dcf952831da1"
 					(reference "#PWR04")
@@
 		(instances
 			(project "Redoubot"
+				(path "/43131b41-4104-4cd6-9c2f-4d5da1687300/089490fe-51aa-455e-8e68-3144de50c1de"
+					(reference "C7")
+					(unit 1)
+				)
 				(path "/43131b41-4104-4cd6-9c2f-4d5da1687300/b7c7d3a9-6fc5-4331-a1be-dcf952831da1"
 					(reference "C2")
@@
 		(instances
 			(project "Redoubot"
+				(path "/43131b41-4104-4cd6-9c2f-4d5da1687300/089490fe-51aa-455e-8e68-3144de50c1de"
+					(reference "#PWR022")
+					(unit 1)
+				)
 				(path "/43131b41-4104-4cd6-9c2f-4d5da1687300/b7c7d3a9-6fc5-4331-a1be-dcf952831da1"
 					(reference "#PWR011")

Commit message: simply added the JLCPCB Part # as an LCSC field in the component descriptions
Parts:
- U2: LCSC (none) -> C50506
Changed lines of the file:
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@@
+			)
+		)
+		(property "LCSC" "C50506"
+			(at 104.14 54.61 0)
+			(hide yes)
+			(show_name no)
+			(do_not_autoplace no)
+			(effects
+				(font
+					(size 1.27 1.27)
+				)
 			)
 		)

Commit message: Added footprints for capacitors
Parts:
- C1: footprint (none) -> Capacitor_SMD:C_0402_1005Metric
- C2: footprint (none) -> Capacitor_SMD:C_0805_2012Metric
- C3: footprint (none) -> Capacitor_SMD:C_0603_1608Metric
Changed lines of the file:
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@@
 			)
 		)
-		(property "Footprint" ""
+		(property "Footprint" "Capacitor_SMD:C_0402_1005Metric"
 			(at 120.65 38.1 0)
 			(hide yes)
@@
 			)
 		)
-		(property "Footprint" ""
+		(property "Footprint" "Capacitor_SMD:C_0603_1608Metric"
 			(at 121.92 48.26 0)
 			(hide yes)
@@
 			)
 		)
-		(property "Footprint" ""
+		(property "Footprint" "Capacitor_SMD:C_0805_2012Metric"
 			(at 113.03 33.02 0)
 			(hide yes)

Commit message: Added the footprints for the resistors, inductors and the crystal
Parts:
- R1: footprint (none) -> Resistor_SMD:R_0805_2012Metric
Changed lines of the file:
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@@
 			)
 		)
-		(property "Footprint" ""
+		(property "Footprint" "Resistor_SMD:R_0805_2012Metric"
 			(at 85.09 50.8 0)
 			(hide yes)

Commit message: feat: added usb_c charging + flashing, added +3.3V generation, added HM10 & DFMini Support, wired everything and modified ioc accordingly
Connections:
- net M+ renamed ML+
- net ML+: no longer U2.2 (AOUT1)
- net M- renamed ML-
- net ML-: no longer U2.4 (AOUT2)
- net PWM_IN1 renamed PWML_IN1
- net PWML_IN1: no longer U2.16 (AIN1)
- net PWM_IN2 renamed PWML_IN2
- net PWML_IN2: no longer U2.15 (AIN2)
- new net MR+: U2.2 (AOUT1)
- new net MR-: U2.4 (AOUT2)
- new net PWMR_IN1: U2.16 (AIN1)
- new net PWMR_IN2: U2.15 (AIN2)
Changed lines of the file:
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@@
-	)
-	(junction
-		(at 120.65 64.77)
-		(diameter 0)
-		(color 0 0 0 0)
 	)
 	(junction
@@
 	)
 	(junction
-		(at 85.09 57.15)
-		(diameter 0)
-		(color 0 0 0 0)
-	)
-	(junction
-		(at 119.38 57.15)
-		(diameter 0)
-		(color 0 0 0 0)
-	)
-	(junction
 		(at 90.17 50.8)
 		(diameter 0)
 		(color 0 0 0 0)
 	)
-	(junction
-		(at 82.55 59.69)
-		(diameter 0)
-		(color 0 0 0 0)
-	)
 	(no_connect
 		(at 116.84 52.07)
@@
 	(wire
 		(pts
-			(xy 116.84 59.69) (xy 120.65 59.69)
+			(xy 116.84 59.69) (xy 129.54 59.69)
 		)
 		(stroke
@@
 	(wire
 		(pts
-			(xy 82.55 64.77) (xy 82.55 59.69)
-		)
-		(stroke
-			(width 0)
-			(type default)
-		)
-	)
-	(wire
-		(pts
-			(xy 91.44 62.23) (xy 85.09 62.23)
-		)
-		(stroke
-			(width 0)
-			(type default)
-		)
-	)
-	(wire
-		(pts
-			(xy 82.55 59.69) (xy 91.44 59.69)
-		)
-		(stroke
-			(width 0)
-			(type default)
-		)
-	)
-	(wire
-		(pts
 			(xy 113.03 30.48) (xy 113.03 29.21)
 		)
@@
 	(wire
 		(pts
-			(xy 120.65 59.69) (xy 120.65 64.77)
-		)
-		(stroke
-			(width 0)
-			(type default)
-		)
-	)
-	(wire
-		(pts
 			(xy 120.65 29.21) (xy 120.65 35.56)
 		)
@@
 	(wire
 		(pts
-			(xy 119.38 57.15) (xy 116.84 57.15)
+			(xy 71.12 64.77) (xy 91.44 64.77)
 		)
 		(stroke
@@
 	(wire
 		(pts
-			(xy 85.09 57.15) (xy 91.44 57.15)
-		)
-		(stroke
-			(width 0)
-			(type default)
-		)
-	)
-	(wire
-		(pts
-			(xy 116.84 62.23) (xy 119.38 62.23)
+			(xy 71.12 57.15) (xy 91.44 57.15)
+		)
+		(stroke
+			(width 0)
+			(type default)
+		)
+	)
+	(wire
+		(pts
+			(xy 116.84 62.23) (xy 129.54 62.23)
 		)
 		(stroke
@@
 	(wire
 		(pts
-			(xy 91.44 64.77) (xy 82.55 64.77)
+			(xy 101.6 26.67) (xy 104.14 26.67)
 		)
 		(stroke
@@
 	(wire
 		(pts
-			(xy 120.65 64.77) (xy 129.54 64.77)
-		)
-		(stroke
-			(width 0)
-			(type default)
-		)
-	)
-	(wire
-		(pts
 			(xy 91.44 52.07) (xy 90.17 52.07)
 		)
@@
 	(wire
 		(pts
-			(xy 71.12 57.15) (xy 85.09 57.15)
+			(xy 71.12 62.23) (xy 91.44 62.23)
 		)
 		(stroke
@@
 	(wire
 		(pts
-			(xy 71.12 59.69) (xy 82.55 59.69)
-		)
-		(stroke
-			(width 0)
-			(type default)
-		)
-	)
-	(wire
-		(pts
-			(xy 85.09 57.15) (xy 85.09 62.23)
+			(xy 71.12 59.69) (xy 91.44 59.69)
 		)
 		(stroke
@@
 	(wire
 		(pts
-			(xy 119.38 62.23) (xy 119.38 57.15)
+			(xy 104.14 26.67) (xy 104.14 29.21)
 		)
 		(stroke
@@
 	(wire
 		(pts
-			(xy 119.38 57.15) (xy 129.54 57.15)
-		)
-		(stroke
-			(width 0)
-			(type default)
-		)
-	)
-	(wire
-		(pts
-			(xy 120.65 64.77) (xy 116.84 64.77)
-		)
-		(stroke
-			(width 0)
-			(type default)
-		)
-	)
-	(wire
-		(pts
-			(xy 104.14 27.94) (xy 104.14 29.21)
-		)
-		(stroke
-			(width 0)
-			(type default)
-		)
-	)
-	(hierarchical_label "M+"
+			(xy 116.84 57.15) (xy 129.54 57.15)
+		)
+		(stroke
+			(width 0)
+			(type default)
+		)
+	)
+	(wire
+		(pts
+			(xy 116.84 64.77) (xy 129.54 64.77)
+		)
+		(stroke
+			(width 0)
+			(type default)
+		)
+	)
+	(hierarchical_label "MR+"
 		(shape output)
 		(at 129.54 57.15 0)
@@
 		)
 	)
-	(hierarchical_label "PWM_IN2"
+	(hierarchical_label "PWML_IN2"
+		(shape input)
+		(at 71.12 64.77 180)
+		(effects
+			(font
+				(size 1.27 1.27)
+			)
+			(justify right)
+		)
+	)
+	(hierarchical_label "MR-"
+		(shape output)
+		(at 129.54 59.69 0)
+		(effects
+			(font
+				(size 1.27 1.27)
+			)
+			(justify left)
+		)
+	)
+	(hierarchical_label "PWMR_IN2"
 		(shape input)
 		(at 71.12 59.69 180)
@@
 	(hierarchical_label "VM"
 		(shape input)
-		(at 104.14 27.94 90)
+		(at 101.6 26.67 180)
 		(effects
 			(font
 				(size 1.27 1.27)
 			)
-			(justify left)
-		)
-	)
-	(hierarchical_label "M-"
+			(justify right)
+		)
+	)
+	(hierarchical_label "PWML_IN1"
+		(shape input)
+		(at 71.12 62.23 180)
+		(effects
+			(font
+				(size 1.27 1.27)
+			)
+			(justify right)
+		)
+	)
+	(hierarchical_label "ML-"
 		(shape output)
 		(at 129.54 64.77 0)
@@
 		)
 	)
-	(hierarchical_label "PWM_IN1"
+	(hierarchical_label "PWMR_IN1"
 		(shape input)
 		(at 71.12 57.15 180)
@@
 			)
 			(justify right)
+		)
+	)
+	(hierarchical_label "ML+"
+		(shape output)
+		(at 129.54 62.23 0)
+		(effects
+			(font
+				(size 1.27 1.27)
+			)
+			(justify left)
 		)
 	)
@@
 		(instances
 			(project "Redoubot"
-				(path "/43131b41-4104-4cd6-9c2f-4d5da1687300/089490fe-51aa-455e-8e68-3144de50c1de"
-					(reference "C8")
-					(unit 1)
-				)
 				(path "/43131b41-4104-4cd6-9c2f-4d5da1687300/b7c7d3a9-6fc5-4331-a1be-dcf952831da1"
 					(reference "C1")
@@
 		(instances
 			(project "Redoubot"
-				(path "/43131b41-4104-4cd6-9c2f-4d5da1687300/089490fe-51aa-455e-8e68-3144de50c1de"
-					(reference "R5")
-					(unit 1)
-				)
 				(path "/43131b41-4104-4cd6-9c2f-4d5da1687300/b7c7d3a9-6fc5-4331-a1be-dcf952831da1"
 					(reference "R1")
@@
 		(instances
 			(project "Redoubot"
-				(path "/43131b41-4104-4cd6-9c2f-4d5da1687300/089490fe-51aa-455e-8e68-3144de50c1de"
-					(reference "#PWR09")
-					(unit 1)
-				)
 				(path "/43131b41-4104-4cd6-9c2f-4d5da1687300/b7c7d3a9-6fc5-4331-a1be-dcf952831da1"
 					(reference "#PWR02")
@@
 		(instances
 			(project "Redoubot"
-				(path "/43131b41-4104-4cd6-9c2f-4d5da1687300/089490fe-51aa-455e-8e68-3144de50c1de"
-					(reference "U3")
-					(unit 1)
-				)
 				(path "/43131b41-4104-4cd6-9c2f-4d5da1687300/b7c7d3a9-6fc5-4331-a1be-dcf952831da1"
 					(reference "U2")
@@
 		(instances
 			(project "Redoubot"
-				(path "/43131b41-4104-4cd6-9c2f-4d5da1687300/089490fe-51aa-455e-8e68-3144de50c1de"
-					(reference "C9")
-					(unit 1)
-				)
 				(path "/43131b41-4104-4cd6-9c2f-4d5da1687300/b7c7d3a9-6fc5-4331-a1be-dcf952831da1"
 					(reference "C3")
@@
 		(instances
 			(project "Redoubot"
-				(path "/43131b41-4104-4cd6-9c2f-4d5da1687300/089490fe-51aa-455e-8e68-3144de50c1de"
-					(reference "#PWR010")
-					(unit 1)
-				)
 				(path "/43131b41-4104-4cd6-9c2f-4d5da1687300/b7c7d3a9-6fc5-4331-a1be-dcf952831da1"
 					(reference "#PWR03")
@@
 		(instances
 			(project "Redoubot"
-				(path "/43131b41-4104-4cd6-9c2f-4d5da1687300/089490fe-51aa-455e-8e68-3144de50c1de"
-					(reference "#PWR023")
-					(unit 1)
-				)
 				(path "/43131b41-4104-4cd6-9c2f-4d5da1687300/b7c7d3a9-6fc5-4331-a1be-dcf952831da1"
 					(reference "#PWR04")
@@
 		(instances
 			(project "Redoubot"
-				(path "/43131b41-4104-4cd6-9c2f-4d5da1687300/089490fe-51aa-455e-8e68-3144de50c1de"
-					(reference "C7")
-					(unit 1)
-				)
 				(path "/43131b41-4104-4cd6-9c2f-4d5da1687300/b7c7d3a9-6fc5-4331-a1be-dcf952831da1"
 					(reference "C2")
@@
 		(instances
 			(project "Redoubot"
-				(path "/43131b41-4104-4cd6-9c2f-4d5da1687300/089490fe-51aa-455e-8e68-3144de50c1de"
-					(reference "#PWR022")
-					(unit 1)
-				)
 				(path "/43131b41-4104-4cd6-9c2f-4d5da1687300/b7c7d3a9-6fc5-4331-a1be-dcf952831da1"
 					(reference "#PWR011")

Commit message: replaced the footprints for resistors with 0402 variants
Parts:
- R1: footprint Resistor_SMD:R_0805_2012Metric -> Resistor_SMD:R_0402_1005Metric
Changed lines of the file:
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@@
 			)
 		)
-		(property "Footprint" "Resistor_SMD:R_0805_2012Metric"
+		(property "Footprint" "Resistor_SMD:R_0402_1005Metric"
 			(at 85.09 50.8 0)
 			(hide yes)

Commit message: fix: Modified the footprints of the capacitors to minimise their size and replaced C2 footprint with an electrolytic capacitor
Parts:
- C2: footprint Capacitor_SMD:C_0805_2012Metric -> Capacitor_SMD:CP_Elec_4x5.4
Changed lines of the file:
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@@
 			)
 		)
-		(property "Footprint" "Capacitor_SMD:C_0805_2012Metric"
+		(property "Footprint" "Capacitor_SMD:CP_Elec_4x5.4"
 			(at 113.03 33.02 0)
 			(hide yes)
