File: Kicad/usb_c.kicad_sch (KiCad schematic)
At the start: 4 parts, among them J13 USB_C_Receptacle_USB2.0_16P, U6 USBLC6-2SC6

Commit message: Feat: Added power LEDs 5v and 3v, Added Jumpers to battery and bms, Added segmentation in connector sheet, Added encoders, Changed page name from motor diver right to motor driver, Redid annotations, Changed output organisation on stm to match new ioc
Parts:
- renumbered J13 to J14, R5 to R20, R6 to R21
Changed lines of the file:
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@@
 		(dnp no)
 		(fields_autoplaced yes)
-		(property "Reference" "J13"
+		(property "Reference" "J14"
 			(at 46.99 22.86 0)
 			(show_name no)
@@
 			(project "Redoubot"
 				(path "/43131b41-4104-4cd6-9c2f-4d5da1687300/7dfaecab-a496-4ad1-bad4-8b5fe60e8651"
-					(reference "J13")
+					(reference "J14")
 					(unit 1)
 				)
@@
 		(dnp no)
 		(fields_autoplaced yes)
-		(property "Reference" "#PWR067"
+		(property "Reference" "#PWR028"
 			(at 88.9 77.47 0)
 			(hide yes)
@@
 			(project "Redoubot"
 				(path "/43131b41-4104-4cd6-9c2f-4d5da1687300/7dfaecab-a496-4ad1-bad4-8b5fe60e8651"
-					(reference "#PWR067")
+					(reference "#PWR028")
 					(unit 1)
 				)
@@
 		(dnp no)
 		(fields_autoplaced yes)
-		(property "Reference" "#PWR065"
+		(property "Reference" "#PWR026"
 			(at 46.99 78.74 0)
 			(hide yes)
@@
 			(project "Redoubot"
 				(path "/43131b41-4104-4cd6-9c2f-4d5da1687300/7dfaecab-a496-4ad1-bad4-8b5fe60e8651"
-					(reference "#PWR065")
+					(reference "#PWR026")
 					(unit 1)
 				)
@@
 		(dnp no)
 		(fields_autoplaced yes)
-		(property "Reference" "R6"
+		(property "Reference" "R21"
 			(at 69.85 34.29 90)
 			(hide yes)
@@
 			(project "Redoubot"
 				(path "/43131b41-4104-4cd6-9c2f-4d5da1687300/7dfaecab-a496-4ad1-bad4-8b5fe60e8651"
-					(reference "R6")
+					(reference "R21")
 					(unit 1)
 				)
@@
 		(dnp no)
 		(fields_autoplaced yes)
-		(property "Reference" "R5"
+		(property "Reference" "R20"
 			(at 69.85 29.21 90)
 			(hide yes)
@@
 			(project "Redoubot"
 				(path "/43131b41-4104-4cd6-9c2f-4d5da1687300/7dfaecab-a496-4ad1-bad4-8b5fe60e8651"
-					(reference "R5")
+					(reference "R20")
 					(unit 1)
 				)
@@
 		(dnp no)
 		(fields_autoplaced yes)
-		(property "Reference" "#PWR066"
+		(property "Reference" "#PWR027"
 			(at 83.82 36.83 0)
 			(hide yes)
@@
 			(project "Redoubot"
 				(path "/43131b41-4104-4cd6-9c2f-4d5da1687300/7dfaecab-a496-4ad1-bad4-8b5fe60e8651"
-					(reference "#PWR066")
-					(unit 1)
-				)
+					(reference "#PWR027")
+					(unit 1)
+				)

Commit message: feat: electrical schematic validated
Parts:
- removed J14: USB_C_Receptacle_USB2.0_16P, Connector_USB:USB_C_Receptacle_GCT_USB4105-xx-A_16P_TopMnt_Horizontal, symbol Connector:USB_C_Receptacle_USB2.0_16P
- removed R20, R21: 5.1k, Resistor_SMD:R_0402_1005Metric, symbol Device:R_Small
- removed U6: USBLC6-2SC6, Package_TO_SOT_SMD:SOT-23-6, symbol Power_Protection:USBLC6-2SC6
Connections:
- no-connect marks 2 -> 0
