File: Kicad/stm32.kicad_sch (KiCad schematic)
At the start: 15 parts, among them J15 Conn_ST_STDC14, U1 STM32G431RBTx, Y1 8MHz

Commit message: feat: added the footprints for new components and started assigning the JLCPCB part numbers
Parts:
- C1, C2: JLCPCB Part # (none) -> C1562
- C19, C20, C21, C22, C25, C27: JLCPCB Part # (none) -> C1525
- C23: JLCPCB Part # (none) -> C23733
- C24: JLCPCB Part # (none) -> C15195
- C26, C28: JLCPCB Part # (none) -> C52923
Changed lines of the file:
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@@
+			)
+		)
+		(property "JLCPCB Part #" "C1525"
+			(at 72.39 43.18 0)
+			(hide yes)
+			(show_name no)
+			(do_not_autoplace no)
+			(effects
+				(font
+					(size 1.27 1.27)
+				)
 			)
 		)
@@
 			)
 		)
+		(property "JLCPCB Part #" "C52923"
+			(at 129.54 33.02 0)
+			(hide yes)
+			(show_name no)
+			(do_not_autoplace no)
+			(effects
+				(font
+					(size 1.27 1.27)
+				)
+			)
+		)
 		(pin "2"
 		)
@@
 			)
 		)
+		(property "JLCPCB Part #" "C52923"
+			(at 63.5 43.18 0)
+			(hide yes)
+			(show_name no)
+			(do_not_autoplace no)
+			(effects
+				(font
+					(size 1.27 1.27)
+				)
+			)
+		)
 		(pin "2"
 		)
@@
 			)
 		)
+		(property "JLCPCB Part #" "C1525"
+			(at 68.58 55.88 0)
+			(hide yes)
+			(show_name no)
+			(do_not_autoplace no)
+			(effects
+				(font
+					(size 1.27 1.27)
+				)
+			)
+		)
 		(pin "2"
 		)
@@
 			)
 		)
+		(property "JLCPCB Part #" "C15195"
+			(at 120.65 33.02 0)
+			(hide yes)
+			(show_name no)
+			(do_not_autoplace no)
+			(effects
+				(font
+					(size 1.27 1.27)
+				)
+			)
+		)
 		(pin "2"
 		)
@@
 			)
 		)
+		(property "JLCPCB Part #" "C1525"
+			(at 76.2 31.75 0)
+			(hide yes)
+			(show_name no)
+			(do_not_autoplace no)
+			(effects
+				(font
+					(size 1.27 1.27)
+				)
+			)
+		)
 		(pin "2"
 		)
@@
 			)
 		)
+		(property "JLCPCB Part #" "C23733"
+			(at 40.64 31.75 0)
+			(hide yes)
+			(show_name no)
+			(do_not_autoplace no)
+			(effects
+				(font
+					(size 1.27 1.27)
+				)
+			)
+		)
 		(pin "2"
 		)
@@
 			)
 		)
+		(property "JLCPCB Part #" "C1525"
+			(at 67.31 31.75 0)
+			(hide yes)
+			(show_name no)
+			(do_not_autoplace no)
+			(effects
+				(font
+					(size 1.27 1.27)
+				)
+			)
+		)
 		(pin "2"
 		)
@@
 		(property "Description" "Unpolarized capacitor"
 			(at 35.56 73.66 0)
+			(hide yes)
+			(show_name no)
+			(do_not_autoplace no)
+			(effects
+				(font
+					(size 1.27 1.27)
+				)
+			)
+		)
+		(property "JLCPCB Part #" "C1562 "
+			(at 35.56 73.66 90)
 			(hide yes)
 			(show_name no)
@@
 			)
 		)
+		(property "JLCPCB Part #" "C1525"
+			(at 58.42 31.75 0)
+			(hide yes)
+			(show_name no)
+			(do_not_autoplace no)
+			(effects
+				(font
+					(size 1.27 1.27)
+				)
+			)
+		)
 		(pin "2"
 		)
@@
 			)
 		)
+		(property "JLCPCB Part #" "C1562 "
+			(at 35.56 53.34 90)
+			(hide yes)
+			(show_name no)
+			(do_not_autoplace no)
+			(effects
+				(font
+					(size 1.27 1.27)
+				)
+			)
+		)
 		(pin "1"
 		)
@@
 			(hide yes)
 			(show_name no)
+			(do_not_autoplace no)
+			(effects
+				(font
+					(size 1.27 1.27)
+				)
+			)
+		)
+		(property "JLCPCB Part #" "C1525"
+			(at 49.53 31.75 0)
+			(hide yes)
+			(show_name no)

Commit message: chore: redid placement from the ground up
Connections:
- net USB_DM: no longer names the net of U1.45 (PA11)
- net USB_DP: no longer names the net of U1.46 (PA12)
- no-connect marks 18 -> 20
Changed lines of the file:
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@@
+	)
+	(no_connect
+		(at 113.03 80.01)
 	)
 	(no_connect
@@
 	)
 	(no_connect
+		(at 113.03 82.55)
+	)
+	(no_connect
 		(at 113.03 90.17)
 	)
@@
 	(wire
 		(pts
-			(xy 113.03 82.55) (xy 133.35 82.55)
-		)
-		(stroke
-			(width 0)
-			(type default)
-		)
-	)
-	(wire
-		(pts
 			(xy 113.03 59.69) (xy 133.35 59.69)
 		)
@@
 		(pts
 			(xy 29.21 63.5) (xy 25.4 63.5)
-		)
-		(stroke
-			(width 0)
-			(type default)
-		)
-	)
-	(wire
-		(pts
-			(xy 113.03 80.01) (xy 133.35 80.01)
 		)
 		(stroke
@@
 		)
 	)
-	(hierarchical_label "USB_DP"
-		(shape input)
-		(at 133.35 82.55 0)
-		(effects
-			(font
-				(size 1.27 1.27)
-			)
-			(justify left bottom)
-		)
-	)
 	(hierarchical_label "SDA_TOF"
 		(shape input)
@@
 		)
 	)
-	(hierarchical_label "USB_DM"
-		(shape input)
-		(at 133.35 80.01 0)
-		(effects
-			(font
-				(size 1.27 1.27)
-			)
-			(justify left bottom)
-		)
-	)
