File: Kicad/stm32.kicad_sch (KiCad schematic)
At the start: 15 parts, among them J15 Conn_ST_STDC14, U1 STM32G431RBTx, Y1 8MHz

Commit message: Feet: finished wiring pcb
53 errors are normal and can be ignored, but should be fixed. PCB can be shrunk by a decent amount.
Connections:
- net INT_ADA: now also U1.51 (PA15); no longer U1.43 (PA9)
- net PWM1_ML: now also U1.42 (PA8); no longer U1.8 (PC0)
- net PWM1_MR: now also U1.44 (PA10); no longer U1.10 (PC2)
- net PWM2_ML: now also U1.43 (PA9); no longer U1.9 (PC1)
- net PWM2_MR: now also U1.45 (PA11); no longer U1.11 (PC3)

Commit message: chore: finished adding all the JLCPCB part numbers for all the components
Parts:
- U1: JLCPCB Part # (none) -> C431633
Changed lines of the file:
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@@
+			)
+		)
+		(property "JLCPCB Part #" "C431633"
+			(at 95.25 92.71 0)
+			(hide yes)
+			(show_name no)
+			(do_not_autoplace no)
+			(effects
+				(font
+					(size 1.27 1.27)
+				)
 			)
 		)
