File: Kicad/connectors.kicad_sch (KiCad schematic)
At the start: 22 parts, among them J1 HM_10_BLE_Module, J10 VL53L0CXV0DH - TOF, J11 DFPlayer_Left, J12 Speaker, J13 DFPlayer_Right, J3 APDS9960, J4 Neopixel, J5 Motor_Left, J6 Motor_Right, J7 MPU-6050, J8 Servo_Left, J9 Servo_Right

Commit message: Chore: Changements M. Fiack
Parts:
- J5, J6: footprint Connector_JST:JST_XH_B6B-XH-AM_1x06_P2.50mm_Vertical -> Connector_JST:JST_XH_B6B-XH-A_1x06_P2.50mm_Vertical
Changed lines of the file:
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@@
 			)
 		)
-		(property "Footprint" "Connector_JST:JST_XH_B6B-XH-AM_1x06_P2.50mm_Vertical"
+		(property "Footprint" "Connector_JST:JST_XH_B6B-XH-A_1x06_P2.50mm_Vertical"
 			(at 73.66 35.56 0)
 			(hide yes)
@@
 			)
 		)
-		(property "Footprint" "Connector_JST:JST_XH_B6B-XH-AM_1x06_P2.50mm_Vertical"
+		(property "Footprint" "Connector_JST:JST_XH_B6B-XH-A_1x06_P2.50mm_Vertical"
 			(at 73.66 55.88 0)
 			(hide yes)
