File: Kicad/drivers.kicad_sch (KiCad schematic)
At the start: 7 parts, among them U5 DRV8833PWP

Commit message: chore: finished adding all the JLCPCB part numbers for all the components
Parts:
- R19, R22: JLCPCB Part # (none) -> C160920
- U5: JLCPCB Part # (none) -> C50506
Changed lines of the file:
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@@
+			)
+		)
+		(property "JLCPCB Part #" "C160920"
+			(at 85.09 48.26 90)
+			(hide yes)
+			(show_name no)
+			(do_not_autoplace no)
+			(effects
+				(font
+					(size 1.27 1.27)
+				)
 			)
 		)
@@
 			)
 		)
+		(property "JLCPCB Part #" "C160920"
+			(at 85.09 53.34 90)
+			(hide yes)
+			(show_name no)
+			(do_not_autoplace no)
+			(effects
+				(font
+					(size 1.27 1.27)
+				)
+			)
+		)
 		(pin "1"
 		)
@@
 			(at 104.14 54.61 0)
 			(hide yes)
+			(show_name no)
+			(do_not_autoplace no)
+			(effects
+				(font
+					(size 1.27 1.27)
+				)
+			)
+		)
+		(property "JLCPCB Part #" "C50506"
+			(at 104.14 54.61 0)
+			(hide yes)
