File: Kicad/power_management.kicad_sch (KiCad schematic)
At the start: 50 parts, among them J14 USB_C_Receptacle_USB2.0_16P, J2 Connecteur batterie, Q1 DMP1045UQ-7, U2 LD39050PU33R, U3 BQ25896RTWR, U4 BQ27220YZFR, U7 DMN313DLT-7, U8 MMDT2907A-7-F

Commit message: chore: finished adding all the JLCPCB part numbers for all the components
Parts:
- D3: JLCPCB Part # C5756798 -> C965804
- L1: JLCPCB Part # (none) -> C42193
- Q1: JLCPCB Part # (none) -> C706746
- R1, R12, R13, R14, R17, R3: JLCPCB Part # (none) -> C25744
- R10, R9: JLCPCB Part # (none) -> C25879
- R11, R4: JLCPCB Part # (none) -> C25741
- R15: JLCPCB Part # (none) -> C11702
- R16, R6: JLCPCB Part # (none) -> C25117
- R18: JLCPCB Part # (none) -> C105362
- R2: JLCPCB Part # (none) -> C25076
- R20, R21: JLCPCB Part # (none) -> C25905
- R5, R7: JLCPCB Part # (none) -> C25867
- R8: JLCPCB Part # (none) -> C25900
- U2: JLCPCB Part # (none) -> C132827
- U3: JLCPCB Part # (none) -> C181475
- U4: JLCPCB Part # (none) -> C528617
- U7: JLCPCB Part # (none) -> C155524
- U8: JLCPCB Part # (none) -> C460232
