File: Kicad/power_management.kicad_sch (KiCad schematic)
At the start: 50 parts, among them J14 USB_C_Receptacle_USB2.0_16P, J2 Connecteur batterie, Q1 DMP1045UQ-7, U2 LD39050PU33R, U3 BQ25896RTWR, U4 BQ27220YZFR, U7 DMN313DLT-7, U8 MMDT2907A-7-F

Commit message: Feat : Finished wiring pcb
shrunk pcb and fixed issues
Parts:
- U4: footprint footprints_BQ27:YZF9_TEX -> Package_BGA:BGA-9_1.6x1.6mm_Layout3x3_P0.5mm
Changed lines of the file:
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@@
 			)
 		)
-		(property "Footprint" "footprints_BQ27:YZF9_TEX"
+		(property "Footprint" "Package_BGA:BGA-9_1.6x1.6mm_Layout3x3_P0.5mm"
 			(at 200.66 39.37 0)
 			(hide yes)
