File: Kicad/_restore_backup_2026-10-07T09-01-36-292/Redoubot.kicad_pcb (KiCad board)
At the start: 4 copper layers, 98 parts, among them J1 HM_10_BLE_Module, J10 VL53L0CXV0DH - TOF, J11 DFPlayer_Left, J12 Speaker, J13 DFPlayer_Right, J14 USB_C_Receptacle_USB2.0_16P, J15 Conn_ST_STDC14, J2 Connecteur batterie, J3 APDS9960, J4 Neopixel, J5 Motor_Left, J6 Motor_Right, J7 MPU-6050, J8 Servo_Left, J9 Servo_Right, Q1 DMP1045UQ-7, U1 STM32G431RBTx, U2 LD39050PU33R, U3 BQ25896RTWR, U4 BQ27220YZFR, U5 DRV8833PWP, U7 DMN313DLT-7, U8 MMDT2907A-7-F, Y1 8MHz

Commit message: feat: placed the power block and started routing
Parts:
- moved R8 100.5 mm to (208.3, 20.4)
- moved U3 100.2 mm to (223.3, 33.7)
- moved JP5 98.1 mm to (218.9, 41.8), turned to 0 degrees
- moved C6 95.7 mm to (214.7, 30.7)
- moved R5 93.3 mm to (205.4, 28.4)
- moved L1 90.7 mm to (214.9, 24.2), turned to 0 degrees
- moved C9 90.7 mm to (214.7, 35.7), turned to 0 degrees
- moved C7 89.9 mm to (214.7, 33.2)
- moved R13 89.7 mm to (208.3, 30.4), turned to 0 degrees
- moved R7 89.1 mm to (205.4, 32.4)
- moved R6 88.9 mm to (205.4, 30.4)
- moved R12 88.9 mm to (208.3, 28.4)
- moved R9 88.6 mm to (209.1, 46.0)
- moved D1 88.6 mm to (206.6, 46.0)
- moved C10 87.2 mm to (214.7, 38.2), turned to 0 degrees
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Connections:
- C3 pad 1: GND -> Net-(JP1-A)
- C3 pad 2: Net-(JP1-A) -> GND
Routing:
- net VBUS: track 27.7 -> 0.00 mm
- net +5V: track 23.7 -> 0.00 mm, vias 1 -> 0
- net +3.3V: track 20.7 -> 0.00 mm, vias 3 -> 0
- net VCC: track 19.4 -> 0.00 mm
- net /Power_management/BAT_CHG: track 18.3 -> 0.00 mm
- net Net-(JP1-A): track 7.92 -> 0.00 mm
- net Net-(C7-Pad2): track 7.90 -> 0.00 mm
- net Net-(U3-STAT): track 7.14 -> 0.00 mm
- net Net-(U3-OTG_IUSB): track 6.29 -> 0.00 mm
- net /SDA_BAT: track 5.39 -> 0.00 mm, vias 2 -> 0
- net Net-(JP5-A): track 5.08 -> 0.00 mm
- net Net-(U8-C2): track 4.69 -> 0.00 mm
- net /SCL_BAT: track 4.46 -> 0.00 mm, vias 2 -> 0
- net Net-(U3-PG_N): track 4.35 -> 0.00 mm
- net /Power_management/BAT: track 4.18 -> 0.00 mm
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