File: Kicad/_restore_backup_2026-10-07T09-48-47-287/Redoubot.kicad_pcb (KiCad board)
At the start: 4 copper layers, 98 parts, among them J1 HM_10_BLE_Module, J10 VL53L0CXV0DH - TOF, J11 DFPlayer_Left, J12 Speaker, J13 DFPlayer_Right, J14 USB_C_Receptacle_USB2.0_16P, J15 Conn_ST_STDC14, J2 Connecteur batterie, J3 APDS9960, J4 Neopixel, J5 Motor_Left, J6 Motor_Right, J7 MPU-6050, J8 Servo_Left, J9 Servo_Right, Q1 DMP1045UQ-7, U1 STM32G431RBTx, U2 LD39050PU33R, U3 BQ25896RTWR, U4 BQ27220YZFR, U5 DRV8833PWP, U7 DMN313DLT-7, U8 MMDT2907A-7-F, Y1 8MHz

Commit message: feat: placed the power block and started routing
Parts:
- moved C16 80.5 mm to (233.5, 118.0), turned to 0 degrees
- moved R14 76.2 mm to (114.3, 25.5), turned to 0 degrees
- moved R17 75.5 mm to (114.3, 26.5), turned to 0 degrees
- moved U4 73.0 mm to (116.3, 26.6), turned to 0 degrees
- moved R18 71.6 mm to (116.0, 29.3), turned to 180 degrees
- moved C14 71.5 mm to (117.9, 25.9), turned to 90 degrees
- moved C13 70.5 mm to (119.1, 25.3), turned to 90 degrees
- moved C15 69.9 mm to (118.4, 27.3), turned to 0 degrees
- moved C29 66.8 mm to (226.5, 118.0), turned to 90 degrees
- moved C17 63.3 mm to (224.3, 119.0), turned to -90 degrees
- moved C18 63.2 mm to (224.8, 117.0), turned to 0 degrees
- moved U5 54.3 mm to (219.8, 118.1), turned to 0 degrees
- moved C3 43.5 mm to (103.0, 48.6)
- moved C4 43.5 mm to (103.0, 51.6)
- moved JP1 43.5 mm to (105.2, 48.4)
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Connections:
- C3 pad 1: GND -> Net-(JP1-A)
- C3 pad 2: Net-(JP1-A) -> GND
Routing:
- net VBUS: track 27.7 -> 0.00 mm
- net +5V: track 23.7 -> 0.00 mm, vias 1 -> 0
- net +3.3V: track 20.7 -> 0.00 mm, vias 3 -> 0
- net VCC: track 19.4 -> 0.00 mm
- net /Power_management/BAT_CHG: track 18.3 -> 0.00 mm
- net Net-(JP1-A): track 7.92 -> 0.00 mm
- net Net-(C7-Pad2): track 7.90 -> 0.00 mm
- net Net-(U3-STAT): track 7.14 -> 0.00 mm
- net Net-(U3-OTG_IUSB): track 6.29 -> 0.00 mm
- net /SDA_BAT: track 5.39 -> 0.00 mm, vias 2 -> 0
- net Net-(U8-C2): track 4.69 -> 0.00 mm
- net /SCL_BAT: track 4.46 -> 0.00 mm, vias 2 -> 0
- net Net-(U3-PG_N): track 4.35 -> 0.00 mm
- net /Power_management/BAT: track 4.18 -> 0.00 mm
- net Net-(U5-BISEN): track 4.12 -> 0.00 mm
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